File: pcb/RTC DS3231/_autosave-RTC DS3231.sch (KiCad schematic (older format))
At the start: 14 parts, among them J101 Conn_01x06_Male, J102 Conn_01x04_Male, U101 DS3231M, U102 AT24CS32-SSHM

Commit message: Modified folders.
Parts:
- BT101: footprint (none) -> Battery:BatteryHolder_Keystone_1058_1x2032
- D101: footprint (none) -> LED_SMD:LED_0402_1005Metric
- D102: footprint (none) -> Diode_SMD:D_0805_2012Metric
- R101, R102: footprint (none) -> Resistor_SMD:R_0805_2012Metric
- RN101, RN102: footprint Resistor_THT:R_Array_SIP5 -> Resistor_SMD:R_Array_Concave_4x0603
Changed lines of the file:
@@
 F 0 "BT101" H 9518 3696 50  0000 L CNN
 F 1 "Battery_Cell" H 9518 3605 50  0000 L CNN
-F 2 "" V 9400 3660 50  0001 C CNN
+F 2 "Battery:BatteryHolder_Keystone_1058_1x2032" V 9400 3660 50  0001 C CNN
 F 3 "~" V 9400 3660 50  0001 C CNN
 	1    9400 3600
@@
 F 0 "RN102" H 6688 2296 50  0000 L CNN
 F 1 "4.7K" H 6688 2205 50  0000 L CNN
-F 2 "Resistor_THT:R_Array_SIP5" V 6775 2250 50  0001 C CNN
+F 2 "Resistor_SMD:R_Array_Concave_4x0603" V 6775 2250 50  0001 C CNN
 F 3 "http://www.vishay.com/docs/31509/csc.pdf" H 6500 2250 50  0001 C CNN
 	1    6500 2250
@@
 F 0 "R101" H 8870 2596 50  0000 L CNN
 F 1 "1k" H 8870 2505 50  0000 L CNN
-F 2 "" V 8730 2550 50  0001 C CNN
+F 2 "Resistor_SMD:R_0805_2012Metric" V 8730 2550 50  0001 C CNN
 F 3 "~" H 8800 2550 50  0001 C CNN
 	1    8800 2550
@@
 F 0 "D101" V 8839 2882 50  0000 R CNN
 F 1 "LED" V 8748 2882 50  0000 R CNN
-F 2 "" H 8800 3000 50  0001 C CNN
+F 2 "LED_SMD:LED_0402_1005Metric" H 8800 3000 50  0001 C CNN
 F 3 "~" H 8800 3000 50  0001 C CNN
 	1    8800 3000
@@
 F 0 "D102" V 9446 2920 50  0000 R CNN
 F 1 "D" V 9355 2920 50  0000 R CNN
-F 2 "" H 9400 3000 50  0001 C CNN
+F 2 "Diode_SMD:D_0805_2012Metric" H 9400 3000 50  0001 C CNN
 F 3 "~" H 9400 3000 50  0001 C CNN
 	1    9400 3000
@@
 F 0 "R102" H 9470 2596 50  0000 L CNN
 F 1 "200" H 9470 2505 50  0000 L CNN
-F 2 "" V 9330 2550 50  0001 C CNN
+F 2 "Resistor_SMD:R_0805_2012Metric" V 9330 2550 50  0001 C CNN
 F 3 "~" H 9400 2550 50  0001 C CNN
 	1    9400 2550
@@
 F 0 "RN101" H 4538 4646 50  0000 L CNN
 F 1 "4.7K" H 4538 4555 50  0000 L CNN
-F 2 "Resistor_THT:R_Array_SIP5" V 4625 4600 50  0001 C CNN
+F 2 "Resistor_SMD:R_Array_Concave_4x0603" V 4625 4600 50  0001 C CNN
 F 3 "http://www.vishay.com/docs/31509/csc.pdf" H 4350 4600 50  0001 C CNN
 	1    4350 4600
