File: pcb/RTC DS3231/RTC DS3231.sch (KiCad schematic (older format))
At the start: 22 parts, among them J101 Conn_01x06_Male, J102 Conn_01x04_Male, U101 DS3231M, U102 AT24CS32-SSHM

Commit message: Deleted images and updated schematic.
Parts:
- BT101: Codigo Mouser (none) -> 710-79548211
- U101: Codigo Mouser (none) -> 700-DS3231M+TRL
- U102: Codigo Mouser (none) -> 556-AT24CS32-SSHM-B
Other:
- moved on the sheet: BT101, C101, C102, D101, D102, FID101, FID102, FID103, H101, H102, H103, J101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

Commit message: Ruteos PCB.
Parts:
- C101, C102: footprint Capacitor_SMD:C_0201_0603Metric -> Capacitor_SMD:C_0805_2012Metric
- D101: footprint LED_SMD:LED_0402_1005Metric -> LED_SMD:LED_0805_2012Metric_Castellated
- RN101, RN102: symbol Device:R_Network04_US -> Device:R_Pack04
Connections:
- net 32KHZ: now also RN102.4 (R4.1); no longer RN102.5 (R4)
- net SCL: now also RN102.2 (R2.1); no longer RN102.3 (R2)
- net SDA: now also RN102.1 (R1.1); no longer RN102.2 (R1)
- net SQW: now also RN102.3 (R3.1); no longer RN102.4 (R3)
- net VCC: now also RN101.5 (R4.2), RN101.6 (R3.2), RN101.7 (R2.2), RN101.8 (R1.2), RN102.5 (R4.2), RN102.6 (R3.2), RN102.7 (R2.2), RN102.8 (R1.2); no longer RN101.1 (common), RN102.1 (common)
- net at JP101.2, U102.1 (A0): now also RN101.4 (R4.1); no longer RN101.5 (R4)
- net at JP102.2, U102.2 (A1): now also RN101.3 (R3.1); no longer RN101.4 (R3)
- net at JP103.2, U102.3 (A2): now also RN101.2 (R2.1); no longer RN101.3 (R2)
