File: pcb/RTC DS3231/RTC DS3231.kicad_pcb (KiCad board)
At the start: 2 copper layers, 42 x 24.5 mm, 22 parts, among them J101 Conn_01x06_Male, J102 Conn_01x04_Male, U101 DS3231M, U102 AT24CS32-SSHM

Commit message: Silks.
Se acomodaron y agregaron las serigrafias en el PCB.
Parts:
- U102: value AT24CS32-SSHM -> AT24CS32
Other:
- board text added: "13-10-2021"
- board text added: "Diseño Argentino"
- board text added: "Matias Meghinasso"
- board text added: "RTC DS3231"
- board text added: "Rev:1"
Changed lines of the file:
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@@
   (general
     (thickness 1.6)
-    (drawings 10)
+    (drawings 15)
     (tracks 195)
     (zones 0)
@@
   (layers
     (0 F.Cu signal)
-    (31 B.Cu signal)
+    (31 B.Cu signal hide)
     (32 B.Adhes user hide)
     (33 F.Adhes user hide)
     (34 B.Paste user hide)
     (35 F.Paste user hide)
-    (36 B.SilkS user hide)
-    (37 F.SilkS user hide)
+    (36 B.SilkS user)
+    (37 F.SilkS user)
     (38 B.Mask user hide)
     (39 F.Mask user hide)
-    (40 Dwgs.User user hide)
+    (40 Dwgs.User user)
     (41 Cmts.User user hide)
     (42 Eco1.User user hide)
-    (43 Eco2.User user)
+    (43 Eco2.User user hide)
     (44 Edge.Cuts user)
     (45 Margin user)
@@
     (47 F.CrtYd user hide)
     (48 B.Fab user hide)
-    (49 F.Fab user hide)
+    (49 F.Fab user)
   )
   (setup
@@
     (pcb_text_size 1.5 1.5)
     (mod_edge_width 0.12)
-    (mod_text_size 1 1)
+    (mod_text_size 0.8 0.8)
     (mod_text_width 0.15)
     (pad_size 1.524 1.524)
@@
     (pad_to_mask_clearance 0)
     (aux_axis_origin 0 0)
-    (visible_elements FFFFFF7F)
+    (visible_elements FFFFF77F)
     (pcbplotparams
       (layerselection 0x010fc_ffffffff)
@@
     (descr "Through hole straight socket strip, 1x04, 2.54mm pitch, single row (from Kicad 4.0.7), script generated")
     (tags "Through hole socket strip THT 1x04 2.54mm single row")
-    (fp_text reference J102 (at 0 -2.77) (layer F.SilkS)
+    (fp_text reference J102 (at -2.25 5.29 90) (layer F.SilkS)
       (effects (font (size 1 1) (thickness 0.15)))
     )
@@
     (tags "resistor array")
     (attr smd)
-    (fp_text reference RN102 (at 0 -2.6) (layer F.SilkS)
+    (fp_text reference RN102 (at 2.7724 -0.1289 90) (layer F.SilkS)
       (effects (font (size 1 1) (thickness 0.15)))
     )
@@
     (tags "solder jumper open")
     (attr virtual)
-    (fp_text reference JP103 (at 0 -1.8 90) (layer F.SilkS)
+    (fp_text reference JP103 (at 1.15 -1.8 90) (layer F.SilkS)
       (effects (font (size 1 1) (thickness 0.15)))
     )
@@
     (tags "solder jumper open")
     (attr virtual)
-    (fp_text reference JP102 (at 0 -1.8 90) (layer F.SilkS)
+    (fp_text reference JP102 (at 1.15 -1.75 90) (layer F.SilkS)
       (effects (font (size 1 1) (thickness 0.15)))
     )
@@
     (tags "solder jumper open")
     (attr virtual)
-    (fp_text reference JP101 (at 0 -1.8 90) (layer F.SilkS)
+    (fp_text reference JP101 (at 1.15 -1.75 90) (layer F.SilkS)
       (effects (font (size 1 1) (thickness 0.15)))
     )
@@
     (tags "LED castellated")
     (attr smd)
-    (fp_text reference D101 (at 0 -1.6) (layer F.SilkS)
+    (fp_text reference D101 (at -3.7924 0) (layer F.SilkS)
       (effects (font (size 1 1) (thickness 0.15)))
     )
@@
     (tags capacitor)
     (attr smd)
-    (fp_text reference C101 (at 0 -1.68) (layer F.SilkS)
+    (fp_text reference C101 (at -3.5224 -0.0251) (layer F.SilkS)
       (effects (font (size 1 1) (thickness 0.15)))
     )
@@
     (tags capacitor)
     (attr smd)
-    (fp_text reference C102 (at 0 -1.68) (layer F.SilkS)
+    (fp_text reference C102 (at -3.5224 -0.1493) (layer F.SilkS)
       (effects (font (size 1 1) (thickness 0.15)))
     )
@@
     (tags diode)
     (attr smd)
-    (fp_text reference D102 (at 0 -1.65 90) (layer F.SilkS)
+    (fp_text reference D102 (at -0.0625 1.75 270) (layer F.SilkS)
       (effects (font (size 1 1) (thickness 0.15)))
     )
@@
     (tags fiducial)
     (attr smd)
-    (fp_text reference FID101 (at 0 -1.5) (layer F.SilkS)
+    (fp_text reference FID101 (at 1.25 1.5) (layer F.SilkS) hide
       (effects (font (size 1 1) (thickness 0.15)))
     )
@@
     (tags fiducial)
     (attr smd)
-    (fp_text reference FID102 (at 0 -1.5) (layer F.SilkS)
+    (fp_text reference FID102 (at 1.25 -1.25) (layer F.SilkS) hide
       (effects (font (size 1 1) (thickness 0.15)))
     )
@@
     (tags fiducial)
     (attr smd)
-    (fp_text reference FID103 (at 0 -1.5) (layer F.SilkS)
+    (fp_text reference FID103 (at -0.25 1.25) (layer F.SilkS) hide
       (effects (font (size 1 1) (thickness 0.15)))
     )
@@
     (tags "mounting hole 2.5mm")
     (attr virtual)
-    (fp_text reference H101 (at 0 -3.5) (layer F.SilkS)
+    (fp_text reference H101 (at 0 3.25) (layer F.SilkS) hide
       (effects (font (size 1 1) (thickness 0.15)))
     )
@@
     (tags "mounting hole 2.5mm")
     (attr virtual)
-    (fp_text reference H102 (at 0 -3.5) (layer F.SilkS)
+    (fp_text reference H102 (at 0 3.25) (layer F.SilkS) hide
       (effects (font (size 1 1) (thickness 0.15)))
     )
@@
     (tags "mounting hole 2.5mm")
     (attr virtual)
-    (fp_text reference H103 (at 0 -3.5) (layer F.SilkS)
+    (fp_text reference H103 (at 0 -3.5) (layer F.SilkS) hide
       (effects (font (size 1 1) (thickness 0.15)))
     )
@@
     (descr "Through hole straight socket strip, 1x06, 2.54mm pitch, single row (from Kicad 4.0.7), script generated")
     (tags "Through hole socket strip THT 1x06 2.54mm single row")
-    (fp_text reference J101 (at 0 -2.77) (layer F.SilkS)
+    (fp_text reference J101 (at 2.25 7.58 90) (layer F.SilkS)
       (effects (font (size 1 1) (thickness 0.15)))
     )
@@
     (tags resistor)
     (attr smd)
-    (fp_text reference R101 (at 0 -1.65) (layer F.SilkS)
+    (fp_text reference R101 (at -3.5224 0.061) (layer F.SilkS)
       (effects (font (size 1 1) (thickness 0.15)))
     )
@@
     (tags "resistor array")
     (attr smd)
-    (fp_text reference RN101 (at 0 -2.6) (layer F.SilkS)
+    (fp_text reference RN101 (at 2.7724 -0.1 90) (layer F.SilkS)
       (effects (font (size 1 1) (thickness 0.15)))
     )
@@
       (effects (font (size 1 1) (thickness 0.15)))
     )
-    (fp_text value AT24CS32-SSHM (at 0 3.4 90) (layer F.Fab)
+    (fp_text value AT24CS32 (at 0 3.4 90) (layer F.Fab)
       (effects (font (size 1 1) (thickness 0.15)))
     )
@@
     )
   )
+  (gr_text "Diseño Argentino" (at 130.5 81.25) (layer B.SilkS)
+    (effects (font (size 0.8 0.8) (thickness 0.15)) (justify mirror))
+  )
+  (gr_text "Matias Meghinasso" (at 130 80) (layer B.SilkS)
+    (effects (font (size 0.8 0.8) (thickness 0.15)) (justify mirror))
+  )
+  (gr_text 13-10-2021 (at 136.5 101.75) (layer B.SilkS)
+    (effects (font (size 0.8 0.8) (thickness 0.15)) (justify mirror))
+  )
+  (gr_text Rev:1 (at 139 100.5) (layer B.SilkS)
+    (effects (font (size 0.8 0.8) (thickness 0.15)) (justify mirror))
+  )
+  (gr_text "RTC DS3231" (at 137 99.25) (layer B.SilkS)
+    (effects (font (size 0.8 0.8) (thickness 0.15)) (justify mirror))
+  )
   (gr_line (start 100.5 102.5) (end 141.5 102.5) (layer Margin) (width 0.15))

Commit message: Anotaciones para fabricación.
Se agregaron las anotaciones para el fabricante del PCB.
Other:
- board text added: "Cantidad de capas: 2 Espesor: 1,6 mm Terminación Superficial: lead-free HASL Componentes: SMD y TH Serigrafía: En ambas caras. Clearance: 0,2 mm Anchos de pista: 0,25 mm Diametro de vias: 0,8 mm Diametro agujeros de Via: 0,4 mm Fabricante de referencia: Meyer Grillas: 0,5 mm y 0,25 mm"
- board text added: "REGLAS DE FABRICACIÓN:"
Changed lines of the file:
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@@
   (general
     (thickness 1.6)
-    (drawings 15)
+    (drawings 17)
     (tracks 195)
     (zones 0)
@@
   (layers
     (0 F.Cu signal)
-    (31 B.Cu signal hide)
+    (31 B.Cu signal)
     (32 B.Adhes user hide)
     (33 F.Adhes user hide)
@@
     (47 F.CrtYd user hide)
     (48 B.Fab user hide)
-    (49 F.Fab user)
+    (49 F.Fab user hide)
   )
   (setup
@@
       (outputformat 1)
       (mirror false)
-      (drillshape 1)
+      (drillshape 0)
       (scaleselection 1)
-      (outputdirectory ""))
+      (outputdirectory "Gerber files/"))
   )
   (net 0 "")
@@
     (fp_line (start 1.88 -0.9) (end 1.88 0.9) (layer F.CrtYd) (width 0.05))
     (fp_line (start 1.88 0.9) (end -1.88 0.9) (layer F.CrtYd) (width 0.05))
-    (pad 2 smd roundrect (at 0.9625 0) (size 1.325 1.3) (layers F.Cu F.Paste F.Mask) (roundrect_rratio 0.192308)
+    (pad 2 smd roundrect (at 0.9625 0) (size 1.325 1.3) (layers F.Cu F.Paste F.Mask) (roundrect_rratio 0.1923076923076923)
       (net 4 "Net-(D101-Pad2)"))
-    (pad 1 smd roundrect (at -0.9625 0) (size 1.325 1.3) (layers F.Cu F.Paste F.Mask) (roundrect_rratio 0.192308)
+    (pad 1 smd roundrect (at -0.9625 0) (size 1.325 1.3) (layers F.Cu F.Paste F.Mask) (roundrect_rratio 0.1923076923076923)
       (net 2 GND))
     (model ${KISYS3DMOD}/LED_SMD.3dshapes/LED_0805_2012Metric_Castellated.wrl
@@
     (fp_line (start 1.68 -0.95) (end 1.68 0.95) (layer F.CrtYd) (width 0.05))
     (fp_line (start 1.68 0.95) (end -1.68 0.95) (layer F.CrtYd) (width 0.05))
-    (pad 2 smd roundrect (at 0.9125 0) (size 1.025 1.4) (layers F.Cu F.Paste F.Mask) (roundrect_rratio 0.243902)
+    (pad 2 smd roundrect (at 0.9125 0) (size 1.025 1.4) (layers F.Cu F.Paste F.Mask) (roundrect_rratio 0.2439014634146341)
       (net 4 "Net-(D101-Pad2)"))
-    (pad 1 smd roundrect (at -0.9125 0) (size 1.025 1.4) (layers F.Cu F.Paste F.Mask) (roundrect_rratio 0.243902)
+    (pad 1 smd roundrect (at -0.9125 0) (size 1.025 1.4) (layers F.Cu F.Paste F.Mask) (roundrect_rratio 0.2439014634146341)
       (net 3 VCC))
     (model ${KISYS3DMOD}/Resistor_SMD.3dshapes/R_0805_2012Metric.wrl
@@
       (effects (font (size 0.5 0.5) (thickness 0.08)))
     )
-    (pad 1 smd roundrect (at -0.9125 0 270) (size 1.025 1.4) (layers F.Cu F.Paste F.Mask) (roundrect_rratio 0.243902)
-      (net 3 VCC))
-    (pad 2 smd roundrect (at 0.9125 0 270) (size 1.025 1.4) (layers F.Cu F.Paste F.Mask) (roundrect_rratio 0.243902)
+    (pad 1 smd roundrect (at -0.9125 0 270) (size 1.025 1.4) (layers F.Cu F.Paste F.Mask) (roundrect_rratio 0.2439014634146341)
+      (net 3 VCC))
+    (pad 2 smd roundrect (at 0.9125 0 270) (size 1.025 1.4) (layers F.Cu F.Paste F.Mask) (roundrect_rratio 0.2439014634146341)
       (net 5 "Net-(D102-Pad2)"))
     (model ${KISYS3DMOD}/Resistor_SMD.3dshapes/R_0805_2012Metric.wrl
@@
     )
   )
+  (gr_text "Cantidad de capas: 2\nEspesor: 1,6 mm\nTerminación Superficial: lead-free HASL\nComponentes: SMD y TH\nSerigrafía: En ambas caras.\nClearance: 0,2 mm\nAnchos de pista: 0,25 mm\nDiametro de vias: 0,8 mm\nDiametro agujeros de Via: 0,4 mm\nFabricante de referencia: Meyer\nGrillas: 0,5 mm y 0,25 mm\n" (at 97.282 117.094) (layer Dwgs.User)
+    (effects (font (size 1 1) (thickness 0.15)) (justify left))
+  )
+  (gr_text "REGLAS DE FABRICACIÓN:" (at 105.5 107.25) (layer Dwgs.User)
+    (effects (font (size 1 1) (thickness 0.15)))
+  )
   (gr_text "Diseño Argentino" (at 130.5 81.25) (layer B.SilkS)
